Commit message: add laser sensor

File: src/urdf_tutorial/urdf/09-mybot.urdf.xacro (robot description, xacro)
@@ -105,3 +105,11 @@
     <origin xyz="0 0 ${bodylen-0.2}"/>
   </joint>
+  <sensor name="laser scanner" update_rate="20">
+    <parent link="head"/>
+    <origin xyz="0 0 ${bodylen+width-0.2}" rpy="0 0 0"/>
+    <ray>
+      <horizontal samples="100" resolution="1" min_angle="-1.5708" max_angle="1.5708"/>
+      <vertical samples="1" resolution="1" min_angle="0" max_angle="0"/>
+    </ray>
+  </sensor>
 </robot>
